File: lyThuyetMach.kicad_pcb (KiCad board)
At the start: 2 copper layers, 48 x 79 mm, 34 parts, among them J1 USB_C_Receptacle_PowerOnly_6P, J2 Voltage_Booster, J4 Out_LED, Q1 BC547, Q2 BC547, Q3 BC547, Q4 BC547, Q5 BC547, Q6 BC547, Q7 TIP122, SW1 SW_SPDT, SW2 SW_SPDT

Commit message: Add files via upload
Parts:
- removed D3: LED, LED_THT:LED_D5.0mm_FlatTop
- removed Q4, Q5, Q6: BC547, Package_TO_SOT_THT:TO-92_Inline
- removed Q7: TIP122, Package_TO_SOT_THT:TO-220-3_Vertical
- removed R10, R15: 470, Resistor_THT:R_Axial_DIN0207_L6.3mm_D2.5mm_P10.16mm_Horizontal
- removed R11, R12, R13, R14, R18: 1k, Resistor_THT:R_Axial_DIN0207_L6.3mm_D2.5mm_P10.16mm_Horizontal
- removed R16, R17: 1M, Resistor_THT:R_Axial_DIN0207_L6.3mm_D2.5mm_P10.16mm_Horizontal
- removed R9: 4.7k, Resistor_THT:R_Axial_DIN0207_L6.3mm_D2.5mm_P10.16mm_Horizontal
- added C1: 100n, Capacitor_THT:C_Disc_D5.0mm_W2.5mm_P5.00mm, F.Cu at (116.5, 99.5)
- added J3: Conn_01x02_Pin, Connector_PinHeader_2.54mm:PinHeader_1x02_P2.54mm_Vertical, F.Cu at (130.3, 103.5)
- D2: footprint LED_THT:LED_D5.0mm_FlatTop -> LED_THT:LED_D5.0mm
- J4: value Out_LED -> Conn_01x02_Pin
- Q1: value BC547 -> BC557
- R4: value 0 -> 4.7k; footprint Resistor_SMD:R_0815_2038Metric_Pad1.20x4.05mm_HandSolder -> Resistor_THT:R_Axial_DIN0207_L6.3mm_D2.5mm_P10.16mm_Horizontal
- R5: value 100 -> 4.7k
- R6: value 4.7k -> 1k
- R7: value 0 -> 10k; footprint Resistor_SMD:R_0815_2038Metric_Pad1.20x4.05mm_HandSolder -> Resistor_THT:R_Axial_DIN0207_L6.3mm_D2.5mm_P10.16mm_Horizontal
- R8: value 100 -> 1M
- moved R5 70.0 mm to (145.7, 98.0), turned to 90 degrees
- moved R8 67.9 mm to (152.2, 98.0)
- moved Q3 60.0 mm to (151.0, 81.9), turned to 0 degrees
- moved D1 59.5 mm to (100.2, 99.0), turned to 0 degrees
- moved R4 53.4 mm to (138.2, 98.1), turned to 90 degrees
- moved J4 53.3 mm to (140.5, 103.5), turned to 90 degrees
- moved R3 51.7 mm to (103.9, 93.5), turned to 0 degrees
- moved Q2 48.4 mm to (140.5, 81.9), turned to 0 degrees
- moved J1 48.0 mm to (90.0, 98.7), turned to 0 degrees
- moved J2 46.8 mm to (92.0, 81.5)
- moved R2 43.8 mm to (103.9, 87.0), turned to 0 degrees
- moved Q1 43.6 mm to (130.0, 81.9), turned to 0 degrees
- moved R6 43.5 mm to (122.0, 88.0), turned to -90 degrees
- moved SW2 41.1 mm to (97.5, 81.5), turned to 0 degrees
- moved R1 36.6 mm to (103.9, 81.0), turned to 0 degrees
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Connections:
- J4 pad 1: Net-(J4-Pin_1) -> VCC
- J4 pad 2: VCC -> Net-(J4-Pin_2)
- Q1 pad 1: Net-(D2-K) -> Net-(D2-A)
- Q1 pad 3: SET -> VCC
- Q2 pad 1: Net-(D3-K) -> Net-(Q2-C)
- Q2 pad 2: Net-(Q2-B) -> Net-(J3-Pin_2)
- Q2 pad 3: RESET -> USB_GND
- Q3 pad 1: LED_Toggle -> Net-(J3-Pin_2)
- Q3 pad 2: Net-(Q3-B) -> Net-(J4-Pin_2)
- R4 pad 1: VCC -> Net-(Q1-B)
- R4 pad 2: Net-(Q1-B) -> Net-(Q2-C)
- R5 pad 2: Net-(D2-A) -> Net-(Q1-B)
- R6 pad 1: SET -> Net-(D2-K)
- R7 pad 1: VCC -> Net-(D2-A)
- R7 pad 2: Net-(Q2-B) -> Net-(J3-Pin_2)
- R8 pad 1: VCC -> Net-(J4-Pin_2)
- R8 pad 2: Net-(D3-A) -> USB_GND
Routing:
- net VCC: track 135.4 -> 0.00 mm, vias 2 -> 0
- net LED_Toggle: track 63.6 -> 0.00 mm
- net SET: track 51.9 -> 0.00 mm
- net Net-(Q1-B): track 32.2 -> 0.00 mm
- net NOT_LED_Toggle: track 31.1 -> 0.00 mm
- net USB_VCC: track 29.3 -> 0.00 mm
- net Net-(Q7-B): track 23.2 -> 0.00 mm
- net Net-(J4-Pin_1): track 22.9 -> 0.00 mm
- net RESET: track 22.1 -> 0.00 mm
- net Net-(Q2-B): track 21.8 -> 0.00 mm
- net Net-(J1-CC1): track 17.9 -> 0.00 mm
- net Net-(Q6-B): track 16.0 -> 0.00 mm
- net Net-(D1-A): track 14.8 -> 0.00 mm
- net Net-(J2-Pin_1): track 14.7 -> 0.00 mm
- net Net-(Q5-B): track 12.5 -> 0.00 mm
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- removed copper zone on B.Cu, net USB_GND
Other:
- board outline removed
